File: pcb/livecam/livecam.kicad_pcb (KiCad board)
At the start: 2 copper layers, 44.5 x 42.4 mm, 24 parts, among them J1 Conn_01x02_Male, J2 Conn_01x02_Male

Commit message: Re-generated gerber files with version number
Other:
- board text added: "LiveCam 1.0"
Changed lines of the file:
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@@
   (general
     (thickness 1.6)
-    (drawings 14)
+    (drawings 15)
     (tracks 253)
     (zones 0)
@@
     )
   )
+  (gr_text "LiveCam 1.0" (at 134.41 42.57) (layer B.SilkS)
+    (effects (font (size 1 1) (thickness 0.15)) (justify mirror))
+  )
   (gr_line (start 168.87 55.86) (end 173.2 55.86) (layer F.SilkS) (width 0.12))
   (gr_line (start 168.87 48.23) (end 168.87 55.86) (layer F.SilkS) (width 0.12))
@@
     (effects (font (size 1 1) (thickness 0.15)) (justify mirror))
   )
-  (gr_text circuitjournal.com (at 163.89 42.08) (layer F.SilkS)
-    (effects (font (size 1 1) (thickness 0.15)))
+  (gr_text circuitjournal.com (at 165.37 42.4) (layer B.SilkS)
+    (effects (font (size 1 1) (thickness 0.15)) (justify mirror))
   )
   (gr_text >7V (at 169.29 70.88) (layer F.SilkS)
